File: DSTB1/kicad/altram_68k_r2.kicad_sch (KiCad schematic)
At the start: 36 parts, among them IC1 IS42S16320D-7TL, IC2 SN74CB3T3245PW, IC3 SN74CB3T3245PW, J1 Conn_01x06_Pin, U1 68000D, U2 68000D, U3 XC95144XL-TQ100, U4 LT1129-3.3_SOT223, X1 IQXO-70

Commit message: No DRC fails. All symbols updated. Bit of ground stitching.
Parts:
- IC2, IC3: Description_1 (none) -> Texas Instruments SN74CB3T3245DW, Bus Switch, 8 x 1:1, 2.3 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
Changed lines of the file:
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@@
 			)
 		)
-		(property "Description" ""
+		(property "Description" "Unpolarized capacitor"
 			(at 279.4 128.27 0)
 			(effects
@@
 			)
 		)
+		(property "Description_1" "Texas Instruments SN74CB3T3245DW, Bus Switch, 8 x 1:1, 2.3  3.6 V, 20-Pin SOIC"
+			(at 367.03 176.53 0)
+			(effects
+				(font
+					(size 1.27 1.27)
+				)
+				(justify left)
+				(hide yes)
+			)
+		)
 		(pin "1"
 		)
@@
 			)
 		)
+		(property "Description_1" "Texas Instruments SN74CB3T3245DW, Bus Switch, 8 x 1:1, 2.3  3.6 V, 20-Pin SOIC"
+			(at 367.03 212.09 0)
+			(effects
+				(font
+					(size 1.27 1.27)
+				)
+				(justify left)
+				(hide yes)
+			)
+		)
 		(pin "1"
 		)
@@
 			)
 		)
-		(property "Description" ""
+		(property "Description" "Unpolarized capacitor"
 			(at 312.42 193.04 0)
 			(effects
@@
 			)
 		)
-		(property "Description" ""
+		(property "Description" "CPLD, 144 Macrocells, 3200 Usable Gates"
 			(at 189.23 207.01 0)
 			(effects
@@
 			)
 		)
-		(property "Description" ""
+		(property "Description" "16/32-bit Microprocessor"
 			(at 81.28 215.9 0)
 			(effects
@@
 			)
 		)
-		(property "Description" ""
+		(property "Description" "4 resistor network, parallel topology"
 			(at 392.43 88.9 0)
 			(effects
@@
 			)
 		)
-		(property "Description" ""
+		(property "Description" "4 resistor network, parallel topology"
 			(at 392.43 71.12 0)
 			(effects
@@
 			)
 		)
-		(property "Description" ""
+		(property "Description" "4 resistor network, parallel topology"
 			(at 392.43 53.34 0)
 			(effects
@@
 			)
 		)
-		(property "Description" ""
+		(property "Description" "4 resistor network, parallel topology"
 			(at 392.43 35.56 0)
 			(effects
@@
 			)
 		)
-		(property "Description" ""
+		(property "Description" "Resistor"
 			(at 129.54 255.27 0)
 			(effects
@@
 			)
 		)
-		(property "Description" ""
+		(property "Description" "700mA Micropower Low drop-out regulator, Fixed Output 3.3V, SOT-223"
 			(at 184.15 38.1 0)
 			(effects
@@
 			)
 		)
-		(property "Description" ""
+		(property "Description" "Crystal Clock Oscillator, SMD package 7.5x5.0mm²"
 			(at 180.34 90.17 0)
 			(effects
@@
 			)
 		)
-		(property "Description" ""
+		(property "Description" "Light emitting diode"
 			(at 257.81 213.36 0)
 			(effects
@@
 			)
 		)
-		(property "Description" ""
+		(property "Description" "Resistor"
 			(at 257.81 203.2 0)
 			(effects
@@
 			)
 		)
-		(property "Description" ""
+		(property "Description" "Unpolarized capacitor"
 			(at 238.76 142.24 0)
 			(effects
@@
 			)
 		)
-		(property "Description" ""
+		(property "Description" "Unpolarized capacitor"
 			(at 248.92 142.24 0)
 			(effects
@@
 			)
 		)
-		(property "Description" ""
+		(property "Description" "Unpolarized capacitor"
 			(at 198.12 41.91 0)
 			(effects
@@
 			)
 		)
-		(property "Description" ""
+		(property "Description" "Unpolarized capacitor"
 			(at 165.1 90.17 0)
 			(effects
@@
 			)
 		)
-		(property "Description" ""
+		(property "Description" "Unpolarized capacitor"
 			(at 30.48 152.4 0)
 			(effects
@@
 			)
 		)
-		(property "Description" ""
+		(property "Description" "Unpolarized capacitor"
 			(at 40.64 152.4 0)
 			(effects
@@
 			)
 		)
-		(property "Description" ""
+		(property "Description" "4 resistor network, parallel topology"
 			(at 351.79 86.36 0)
 			(effects
@@
 			)
 		)
-		(property "Description" ""
+		(property "Description" "4 resistor network, parallel topology"
 			(at 351.79 68.58 0)
 			(effects
@@
 			)
 		)
-		(property "Description" ""
+		(property "Description" "4 resistor network, parallel topology"
 			(at 351.79 50.8 0)
 			(effects
@@
 			)
 		)
-		(property "Description" ""
+		(property "Description" "4 resistor network, parallel topology"
 			(at 351.79 33.02 0)
 			(effects
@@
 			)
 		)
-		(property "Description" ""
+		(property "Description" "4 resistor network, parallel topology"
 			(at 351.79 121.92 0)
 			(effects
@@
 			)
 		)
-		(property "Description" ""
+		(property "Description" "4 resistor network, parallel topology"
 			(at 351.79 104.14 0)
 			(effects
@@
 			)
 		)
-		(property "Description" ""
+		(property "Description" "test point"
 			(at 378.46 157.48 0)
 			(effects
@@
 			)
 		)
-		(property "Description" ""
+		(property "Description" "test point"
 			(at 378.46 147.32 0)
 			(effects
@@
 			)
 		)
-		(property "Description" ""
+		(property "Description" "test point"
 			(at 378.46 142.24 0)
 			(effects
@@
 			)
 		)
-		(property "Description" ""
+		(property "Description" "test point"
 			(at 378.46 137.16 0)
 			(effects
@@
 			)
 		)
-		(property "Description" ""
+		(property "Description" "test point"
 			(at 378.46 152.4 0)
 			(effects

Commit message: Adding an inline termination to the clk8 line, just in case.
Parts:
- added R4: 10R, Resistor_SMD:R_0805_2012Metric_Pad1.20x1.40mm_HandSolder, symbol Device:R
Connections:
- net CLK8: now also R4.1; no longer U1.15 (CLK)
- new net CLK_ST: R4.2, U1.15 (CLK)
Changed lines of the file:
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@@
 		)
 	)
+	(wire
+		(pts
+			(xy 38.1 24.13) (xy 55.88 24.13)
+		)
+		(stroke
+			(width 0)
+			(type default)
+		)
+	)
 	(bus
 		(pts
@@
 		)
 	)
+	(label "CLK_ST"
+		(at 55.88 24.13 180)
+		(fields_autoplaced yes)
+		(effects
+			(font
+				(size 1.27 1.27)
+			)
+			(justify right bottom)
+		)
+	)
 	(label "A10"
 		(at 218.44 163.83 0)
@@
 	(global_label "CLK8"
 		(shape output)
-		(at 55.88 24.13 180)
+		(at 30.48 24.13 180)
 		(fields_autoplaced yes)
 		(effects
@@
 		)
 		(property "Intersheetrefs" "${INTERSHEET_REFS}"
-			(at 48.7714 24.13 0)
+			(at 23.3714 24.13 0)
 			(effects
 				(font
@@
 					(unit 1)
 				)
+			)
+		)
+	)
+	(symbol
+		(lib_id "Device:R")
+		(at 34.29 24.13 90)
+		(unit 1)
+		(exclude_from_sim no)
+		(in_bom yes)
+		(on_board yes)
+		(dnp no)
+		(fields_autoplaced yes)
+		(property "Reference" "R4"
+			(at 34.29 18.9695 90)
+			(effects
+				(font
+					(size 1.27 1.27)
+				)
+			)
+		)
+		(property "Value" "10R"
+			(at 34.29 21.3938 90)
+			(effects
+				(font
+					(size 1.27 1.27)
+				)
+			)
+		)
+		(property "Footprint" "Resistor_SMD:R_0805_2012Metric_Pad1.20x1.40mm_HandSolder"
+			(at 34.29 25.908 90)
+			(effects
+				(font
+					(size 1.27 1.27)
+				)
+				(hide yes)
+			)
+		)
+		(property "Datasheet" "~"
+			(at 34.29 24.13 0)
+			(effects
+				(font
+					(size 1.27 1.27)
+				)
+				(hide yes)
+			)
+		)
+		(property "Description" "Resistor"
+			(at 34.29 24.13 0)
+			(effects
+				(font
+					(size 1.27 1.27)
+				)
+				(hide yes)
+			)
+		)
+		(pin "2"
+		)
+		(pin "1"
+		)
+		(instances
+			(project ""
+				(path "/c9a72e4c-f90e-4205-9d40-436bd9db8a4b"
+					(reference "R4")
+					(unit 1)
+				)

Commit message: Rejigged the bottom a bit to provide a better ground plane. Changed to the 1117-3.3 regulator
Parts:
- removed U4: LT1129-3.3_SOT223, Package_TO_SOT_SMD:SOT-223-3_TabPin2, symbol Regulator_Linear:LT1129-3.3_SOT223
- added C8: 100n, Capacitor_SMD:C_0805_2012Metric_Pad1.18x1.45mm_HandSolder, symbol Device:C
- added U4: AMS1117-3.3, Package_TO_SOT_SMD:SOT-223-3_TabPin2, symbol Regulator_Linear:AMS1117-3.3
- C3: renamed from C5; value 100n -> 10u
- C7: renamed from C10; value 10u -> 100n
- R2: footprint Capacitor_SMD:C_0805_2012Metric_Pad1.18x1.45mm_HandSolder -> Resistor_SMD:R_0805_2012Metric_Pad1.20x1.40mm_HandSolder
- renumbered C8 to C1, C4 to C2, C3 to C4, C1 to C5, C7 to C6
Connections:
- net GND: now also C8.1, U4.1 (GND)
- net TP2: now also U3.16 (P16); no longer U3.17 (P17)
- net VCC: now also R3.2, U4.3 (VI)
- net VCC3: now also C8.2, U4.2 (VO); no longer R3.2
- net ~{HLT}: now also U3.17 (P17)
- no-connect marks 9 -> 8
